File: Power.kicad_sch (KiCad schematic)
At the start: 12 parts, among them U3 TPS7A20, U4 TPS7A20

Commit message: MDIX routing done
Connections:
- net 1V1: now also U3.5 (OUT); no longer U3.2 (OUT)
- net 2V5: now also U4.5 (OUT); no longer U4.2 (OUT)
- net GND: now also U3.2 (GND), U4.2 (GND); no longer U3.5 (GND), U4.5 (GND)
