File: pocketbeagle2 revA_241205.kicad_pcb (KiCad board)
At the start: 4 copper layers, 85 parts, among them J1 1840888-1, P1 PMOD_I2S, P2 PMOD_I2S, Q1 BSS138, Q2 BSS138, Q3 BSS138, U1 PocketBeagle2, U2 DP83867IRPAPR, U3 TPS7A20, U4 TPS7A20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

Commit message: Updating pcb
Parts:
- moved TP4 3.48 mm to (212.0, 86.0)
- moved R21 2.00 mm to (208.6, 82.5)
- moved C6 1.75 mm to (205.6, 85.2)
- moved C27 1.38 mm to (205.6, 80.8)
- moved C20 1.38 mm to (205.6, 84.0)
- moved R20 1.35 mm to (209.5, 84.0)
- moved C23 1.14 mm to (188.0, 85.5)
- moved C22 1.00 mm to (205.6, 82.8)
- moved C17 1.00 mm to (205.6, 79.5)
- moved C26 0.76 mm to (205.5, 89.4)
- moved C3 0.43 mm to (188.0, 84.5)
- moved C15 0.43 mm to (187.8, 88.8)
- moved C13 0.26 mm to (205.5, 90.5)
- moved C19 0.25 mm to (187.8, 89.9)
Routing:
- net /Network/LED2: track 14.5 -> 0.00 mm
- net RESET_N: track 0.00 -> 13.3 mm, vias 0 -> 1
- net MDIO0_DIO: track 0.00 -> 9.12 mm
- net MDIO0_MDC: track 0.00 -> 8.79 mm
- net INT_N/PWRDN_N: track 8.54 -> 0.00 mm
- net /Network/LED1: track 11.0 -> 2.59 mm
- net /Network/LED0: track 8.07 -> 0.00 mm
- net /Network/X_IN: track 9.47 -> 12.4 mm
- net /Network/RX_D7: track 0.00 -> 2.92 mm
- net Net-(D3-A): track 1.81 -> 0.00 mm
- net Net-(D3-K): track 22.1 -> 23.7 mm
- added copper zone on In1.Cu, net GND
Other:
- board outline added: 35.3 x 55.3 mm

Commit message: Preparing routing for RGMII and MDI interfaces
Parts:
- moved TP6 9.19 mm to (205.0, 57.0)
- moved TP8 7.08 mm to (188.2, 57.0)
- moved TP7 6.58 mm to (190.5, 57.0)
- moved C33 6.37 mm to (199.8, 56.2), turned to 180 degrees
- moved C31 6.29 mm to (193.8, 56.2), turned to 0 degrees
- moved C30 3.82 mm to (193.5, 62.2), turned to 180 degrees
- moved TP5 2.26 mm to (207.8, 57.8)
- moved R12 2.25 mm to (188.9, 83.8)
- moved R13 1.01 mm to (188.8, 81.5)
- moved C34 0.79 mm to (196.2, 61.8)
- moved C35 0.35 mm to (202.2, 62.2), turned to 180 degrees
- moved R7 0.25 mm to (188.9, 82.8)
- moved C15 0.20 mm to (187.9, 88.6)
- moved C19 0.20 mm to (187.9, 89.8)
Connections:
- U3 pad 2: VDD_1V1 -> GND
- U3 pad 5: GND -> VDD_1V1
- U4 pad 2: VDD_2V5 -> GND
- U4 pad 5: GND -> VDD_2V5
Routing:
- net PMOD2.SDOUT: track 0.00 -> 65.7 mm, vias 0 -> 1
- net MCLK_TOUT: track 1.50 -> 56.1 mm, vias 0 -> 1
- net INT_N/PWRDN_N: track 0.00 -> 27.3 mm, vias 0 -> 1
- net LRCK: track 35.2 -> 60.6 mm, vias 1 -> 2
- net MDIO0_MDC: track 8.79 -> 21.6 mm, vias 0 -> 1
- net RGMII_TX_CTRL: track 0.00 -> 10.7 mm, vias 0 -> 2
- net Net-(U2-RX_CLK): track 0.00 -> 10.0 mm, vias 0 -> 1
- net Net-(U2-TX_D1): track 0.00 -> 9.94 mm, vias 0 -> 1
- net RGMII_RX_CTRL: track 0.00 -> 9.93 mm, vias 0 -> 3
- net Net-(U2-TX_D0): track 0.00 -> 9.66 mm, vias 0 -> 1
- net Net-(U2-RX_D0): track 0.00 -> 9.54 mm, vias 0 -> 1
- net Net-(U2-GTX_CLK): track 0.00 -> 9.33 mm, vias 0 -> 1
- net Net-(U2-RX_D1): track 0.00 -> 9.13 mm, vias 0 -> 1
- net RESET_N: track 13.3 -> 22.2 mm
- net Net-(U2-RX_D2): track 0.00 -> 8.76 mm, vias 0 -> 1
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- added copper zone on F.Cu, net GND
- added copper zone on F.Cu, net VDD_3V3

Commit message: MDIX routing done
Parts:
- removed TP3: TestPoint, TestPoint:TestPoint_Pad_1.0x1.0mm
- moved C15 0.85 mm to (188.0, 89.4)
- moved C19 0.85 mm to (188.0, 90.6)
- moved R5 0.55 mm to (187.6, 78.5)
- moved R6 0.55 mm to (187.6, 77.2)
- moved C25 0.50 mm to (197.2, 93.1)
- moved C7 0.50 mm to (195.2, 93.1)
- moved R24 0.40 mm to (185.9, 82.1)
Connections:
- net Net-(J1-MD0+) renamed /Network/MD0_P
- net Net-(J1-MD0-) renamed /Network/MD0_N
- net Net-(J1-MD1+) renamed /Network/MD1_P
- net Net-(J1-MD1-) renamed /Network/MD1_N
- net Net-(J1-MD2+) renamed /Network/MD2_P
- net Net-(J1-MD2-) renamed /Network/MD2_N
- net Net-(J1-MD3+) renamed /Network/MD3_P
- net Net-(J1-MD3-) renamed /Network/MD3_N
- U1 pad 26: I2C2_SDA -> unconnected-(U1-I2C2.SDA-Pad26)
- U1 pad 28: I2C2_SCL -> unconnected-(U1-I2C2.SCL-Pad28)
- U2 pad 17: Net-(TP3-Pad1) -> unconnected-(U2-VDDA1P8-Pad17)
- U2 pad 64: Net-(TP3-Pad1) -> unconnected-(U2-VDDA1P8-Pad17)
Routing:
- net VDD_2V5: track 0.00 -> 157.9 mm, vias 0 -> 3
- net VDD_3V3: track 2.50 -> 139.7 mm, vias 0 -> 7
- net VDD_1V1: track 0.00 -> 91.6 mm, vias 0 -> 5
- net MDIO0_MDC: track 21.6 -> 56.5 mm, vias 1 -> 2
- net PMOD2.SDOUT: track 65.7 -> 81.9 mm
- net /Network/LED2: track 0.00 -> 14.0 mm
- net /Network/RX_D7: track 1.27 -> 12.9 mm, vias 0 -> 2
- net /Network/MD0_P: track 0.00 -> 9.71 mm
- net /Network/MD2_N: track 0.00 -> 9.66 mm
- net /Network/MD0_N: track 0.00 -> 9.65 mm
- net /Network/MD3_P: track 0.00 -> 9.60 mm
- net /Network/MD3_N: track 0.00 -> 9.54 mm
- net /Network/MD1_P: track 0.00 -> 9.27 mm
- net /Network/MD2_P: track 0.00 -> 9.26 mm
- net /Network/MD1_N: track 0.00 -> 9.22 mm
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- removed copper zone on F.Cu, net GND
- removed copper zone on F.Cu, net VDD_3V3

Commit message: Fully routed PCB, missing fligth time matching on the RGMII
Parts:
- moved R28 0.99 mm to (182.1, 102.5)
- moved D3 0.71 mm to (182.2, 100.7)
- moved C23 0.35 mm to (188.3, 85.6)
- moved C12 0.25 mm to (187.9, 81.8)
Connections:
- J1 pad S2: Net-(J1-SHIELD) -> Net-(J1-SHIELD__1)
- R26 pad 2: Net-(J1-SHIELD) -> Net-(J1-SHIELD__1)
- U1 pad 67: RGMII_TD3 -> RGMII_TD1
- U2 pad 64: unconnected-(U2-VDDA1P8-Pad17) -> unconnected-(U2-VDDA1P8-Pad64)
- U2 pad V: unconnected-(U2-NC-PadV) -> GND
Routing:
- net VDD_3V3: track 139.7 -> 266.6 mm, vias 7 -> 13
- net MCLK_TIN: track 4.18 -> 59.4 mm, vias 2 -> 4
- net RGMII_TX_CLK: track 3.19 -> 49.4 mm
- net GND: track 0.00 -> 37.4 mm, vias 0 -> 14
- net RGMII_RX_CLK: track 2.99 -> 34.2 mm
- net RGMII_TD1: track 1.62 -> 32.2 mm, vias 1 -> 2
- net MDIO0_DIO: track 15.7 -> 44.8 mm, vias 1 -> 3
- net RGMII_RX_CTRL: track 6.50 -> 32.1 mm
- net RGMII_RD0: track 3.14 -> 27.6 mm
- net RGMII_TD2: track 7.69 -> 30.5 mm
- net RGMII_RD1: track 3.45 -> 24.0 mm
- net RGMII_TX_CTRL: track 8.03 -> 26.8 mm
- net RGMII_RD2: track 3.29 -> 21.5 mm
- net RGMII_RD3: track 2.92 -> 18.1 mm
- net RGMII_TD0: track 7.33 -> 22.2 mm
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- added copper zone on B.Cu, net GND
- added copper zone on F.Cu, net GND
- added copper zone on F.Cu, net VDD_1V1
- added copper zone on F.Cu, net VDD_2V5
