File: pocketbeagle2_ethernet_cap.kicad_sch (KiCad schematic)
At the start: 1 part, among them U1 PocketBeagle2

Commit message: Split Power into ldo_1v1 and ldo_2v5 sheets, rename audio sheet
Other:
- sheet Audio renamed audio
- removed sheet Power
- added sheet ldo_1v1 (ldo_1v1.kicad_sch)
- added sheet ldo_2v5 (ldo_2v5.kicad_sch)
- sheet audio: file Audio.kicad_sch -> audio.kicad_sch
Changed lines of the file:
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@@
-	(wire
-		(pts
-			(xy 190.5 146.05) (xy 198.12 146.05)
-		)
-		(stroke
-			(width 0)
-			(type default)
-		)
-	)
 	(wire
 		(pts
@@
 	(wire
 		(pts
-			(xy 190.5 142.24) (xy 198.12 142.24)
-		)
-		(stroke
-			(width 0)
-			(type default)
-		)
-	)
-	(wire
-		(pts
 			(xy 172.72 35.56) (xy 177.8 35.56)
 		)
@@
 	(wire
 		(pts
-			(xy 190.5 149.86) (xy 198.12 149.86)
-		)
-		(stroke
-			(width 0)
-			(type default)
-		)
-	)
-	(wire
-		(pts
 			(xy 224.79 35.56) (xy 219.71 35.56)
 		)
@@
 		(property "Intersheetrefs" "${INTERSHEET_REFS}"
 			(at 161.5705 99.06 0)
-			(effects
-				(font
-					(size 1.27 1.27)
-				)
-				(justify right)
-				(hide yes)
-			)
-		)
-	)
-	(global_label "VDD_3V3"
-		(shape input)
-		(at 190.5 149.86 180)
-		(fields_autoplaced yes)
-		(effects
-			(font
-				(size 1.27 1.27)
-			)
-			(justify right)
-		)
-		(property "Intersheetrefs" "${INTERSHEET_REFS}"
-			(at 179.411 149.86 0)
 			(effects
 				(font
@@
 		)
 	)
-	(global_label "VDD_2V5"
-		(shape output)
-		(at 190.5 146.05 180)
-		(fields_autoplaced yes)
-		(effects
-			(font
-				(size 1.27 1.27)
-			)
-			(justify right)
-		)
-		(property "Intersheetrefs" "${INTERSHEET_REFS}"
-			(at 179.411 146.05 0)
-			(effects
-				(font
-					(size 1.27 1.27)
-				)
-				(justify right)
-				(hide yes)
-			)
-		)
-	)
 	(global_label "RGMII_RX_CLK"
 		(shape input)
@@
 		(property "Intersheetrefs" "${INTERSHEET_REFS}"
 			(at 160.1191 33.02 0)
-			(effects
-				(font
-					(size 1.27 1.27)
-				)
-				(justify right)
-				(hide yes)
-			)
-		)
-	)
-	(global_label "VDD_1V1"
-		(shape output)
-		(at 190.5 142.24 180)
-		(fields_autoplaced yes)
-		(effects
-			(font
-				(size 1.27 1.27)
-			)
-			(justify right)
-		)
-		(property "Intersheetrefs" "${INTERSHEET_REFS}"
-			(at 179.411 142.24 0)
 			(effects
 				(font
@@
 		)
 		(instances
-			(project "pocketbeagle2 revA_241205"
+			(project "pocketbeagle2_ethernet_cap"
 				(path "/82320ebb-b624-4fc9-8d5a-3bc164182d09"
 					(reference "#PWR01")
@@
 		)
 		(instances
-			(project "pocketbeagle2 revA_241205"
+			(project "pocketbeagle2_ethernet_cap"
 				(path "/82320ebb-b624-4fc9-8d5a-3bc164182d09"
 					(reference "U1")
@@
 		)
 		(instances
-			(project "pocketbeagle2 revA_241205"
+			(project "pocketbeagle2_ethernet_cap"
 				(path "/82320ebb-b624-4fc9-8d5a-3bc164182d09"
 					(page "3")
@@
 		)
 	)
-	(sheet
-		(at 198.12 139.7)
-		(size 12.7 12.7)
-		(exclude_from_sim no)
-		(in_bom yes)
-		(on_board yes)
-		(dnp no)
-		(fields_autoplaced yes)
-		(stroke
-			(width 0.1524)
-			(type solid)
-		)
-		(fill
-			(color 0 0 0 0.0000)
-		)
-		(property "Sheetname" "Power"
-			(at 198.12 138.9884 0)
-			(effects
-				(font
-					(size 1.27 1.27)
-				)
-				(justify left bottom)
-			)
-		)
-		(property "Sheetfile" "Power.kicad_sch"
-			(at 198.12 152.9846 0)
-			(effects
-				(font
-					(size 1.27 1.27)
-				)
-				(justify left top)
-			)
-		)
-		(pin "1V1" output
-			(at 198.12 142.24 180)
-			(effects
-				(font
-					(size 1.27 1.27)
-				)
-				(justify left)
-			)
-		)
-		(pin "3V3" input
-			(at 198.12 149.86 180)
-			(effects
-				(font
-					(size 1.27 1.27)
-				)
-				(justify left)
-			)
-		)
-		(pin "2V5" output
-			(at 198.12 146.05 180)
-			(effects
-				(font
-					(size 1.27 1.27)
-				)
-				(justify left)
-			)
-		)
-		(instances
-			(project "pocketbeagle2 revA_241205"
-				(path "/82320ebb-b624-4fc9-8d5a-3bc164182d09"
-					(page "4")
-				)
-			)
-		)
-	)
-	(sheet
+		(sheet
 		(at 180.34 90.17)
 		(size 44.45 34.29)
@@
 			(color 0 0 0 0.0000)
 		)
-		(property "Sheetname" "Audio"
+		(property "Sheetname" "audio"
 			(at 180.34 89.4584 0)
 			(effects
@@
 			)
 		)
-		(property "Sheetfile" "Audio.kicad_sch"
+		(property "Sheetfile" "audio.kicad_sch"
 			(at 180.34 125.0446 0)
 			(effects
@@
 		)
 		(instances
-			(project "pocketbeagle2 revA_241205"
+			(project "pocketbeagle2_ethernet_cap"
 				(path "/82320ebb-b624-4fc9-8d5a-3bc164182d09"
 					(page "2")
@@
 		)
 	)
+	(sheet
+		(at 198.12 138.43)
+		(size 12.7 7.62)
+		(exclude_from_sim no)
+		(in_bom yes)
+		(on_board yes)
+		(dnp no)
+		(fields_autoplaced yes)
+		(stroke
+			(width 0.1524)
+			(type solid)
+		)
+		(fill
+			(color 0 0 0 0.0000)
+		)
+		(property "Sheetname" "ldo_1v1"
+			(at 198.12 137.7184 0)
+			(effects
+				(font
+					(size 1.27 1.27)
+				)
+				(justify left bottom)
+			)
+		)
+		(property "Sheetfile" "ldo_1v1.kicad_sch"
+			(at 198.12 146.76160000000002 0)
+			(effects
+				(font
+					(size 1.27 1.27)
+				)
+				(justify left top)
+			)
+		)
+		(pin "3V3" input
+			(at 198.12 140.97 180)
+			(effects
+				(font
+					(size 1.27 1.27)
+				)
+				(justify right)
+			)
+		)
+		(pin "1V1" output
+			(at 198.12 143.51 180)
+			(effects
+				(font
+					(size 1.27 1.27)
+				)
+				(justify right)
+			)
+		)
+		(instances
+			(project "pocketbeagle2_ethernet_cap"
+				(path "/82320ebb-b624-4fc9-8d5a-3bc164182d09"
+					(page "5")
+				)
+			)
+		)
+	)
+	(sheet
+		(at 198.12 151.13)
+		(size 12.7 7.62)
+		(exclude_from_sim no)
+		(in_bom yes)
+		(on_board yes)
+		(dnp no)
+		(fields_autoplaced yes)
+		(stroke
+			(width 0.1524)
+			(type solid)
+		)
+		(fill
+			(color 0 0 0 0.0000)
+		)
+		(property "Sheetname" "ldo_2v5"
+			(at 198.12 150.4184 0)
+			(effects
+				(font
+					(size 1.27 1.27)
+				)
+				(justify left bottom)
+			)
+		)
+		(property "Sheetfile" "ldo_2v5.kicad_sch"
+			(at 198.12 159.4616 0)
+			(effects
+				(font
+					(size 1.27 1.27)
+				)
+				(justify left top)
+			)
+		)
+		(pin "3V3" input
+			(at 198.12 153.67 180)
+			(effects
+				(font
+					(size 1.27 1.27)
+				)
+				(justify right)
+			)
+		)
+		(pin "2V5" output
+			(at 198.12 156.21 180)
+			(effects
+				(font
+					(size 1.27 1.27)
+				)
+				(justify right)
+			)
+		)
+		(instances
+			(project "pocketbeagle2_ethernet_cap"
+				(path "/82320ebb-b624-4fc9-8d5a-3bc164182d09"
+					(page "6")
+				)
+			)
+		)
+	)
+	(wire
+		(pts
+			(xy 190.5 140.97) (xy 198.12 140.97)
+		)
+		(stroke
+			(width 0)
+			(type default)
+		)
+	)
+	(global_label "VDD_3V3"
+		(shape input)
+		(at 190.5 140.97 180)
+		(effects
+			(font
+				(size 1.27 1.27)
+			)
+			(justify right)
+		)
+	)
+	(wire
+		(pts
+			(xy 190.5 143.51) (xy 198.12 143.51)
+		)
+		(stroke
+			(width 0)
+			(type default)
+		)
+	)
+	(global_label "VDD_1V1"
+		(shape output)
+		(at 190.5 143.51 180)
+		(effects
+			(font
+				(size 1.27 1.27)
+			)
+			(justify right)
+		)
+	)
+	(wire
+		(pts
+			(xy 190.5 153.67) (xy 198.12 153.67)
+		)
+		(stroke
+			(width 0)
+			(type default)
+		)
+	)
+	(global_label "VDD_3V3"
+		(shape input)
+		(at 190.5 153.67 180)
+		(effects
+			(font
+				(size 1.27 1.27)
+			)
+			(justify right)
+		)
+	)
+	(wire
+		(pts
+			(xy 190.5 156.21) (xy 198.12 156.21)
+		)
+		(stroke
+			(width 0)
+			(type default)
+		)
+	)
+	(global_label "VDD_2V5"
+		(shape output)
+		(at 190.5 156.21 180)
+		(effects
+			(font
+				(size 1.27 1.27)
+			)
+			(justify right)
+		)
+	)

Commit message: Migrate root sheet to KL PocketBeagle2 module symbol
Parts:
- U1: footprint Module:BeagleBoard_PocketBeagle -> KL_Footprints:BeagleBoard_PocketBeagle; symbol MCU_Module:PocketBeagle -> KL_Module:PocketBeagle2; Digikey (none) -> TBD; LCSC (none) -> TBD; MPN (none) -> PocketBeagle 2; Mouser (none) -> TBD
Changed lines of the file:
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@@
 	)
 	(symbol
-		(lib_id "MCU_Module:PocketBeagle")
+		(lib_id "KL_Module:PocketBeagle2")
 		(at 67.31 82.55 0)
 		(unit 1)
@@
 			)
 		)
-		(property "Footprint" "Module:BeagleBoard_PocketBeagle"
+		(property "Footprint" "KL_Footprints:BeagleBoard_PocketBeagle"
 			(at 67.31 82.55 0)
 			(effects
@@
 			)
 		)
-		(property "Datasheet" "https://github.com/beagleboard/pocketbeagle/wiki/System-Reference-Manual"
+		(property "Datasheet" "https://docs.beagleboard.org/boards/pocketbeagle-2/"
 			(at 110.49 115.57 0)
 			(effects
@@
 			)
 		)
-		(property "Description" "Singleboard computer with ARM Cortex-A8 1GHz, 512MB RAM"
+		(property "Description" "BeagleBoard.org PocketBeagle 2 host board (AM62x)"
 			(at 67.31 82.55 0)
 			(effects
@@
 			)
 		)
+		(property "MPN" "PocketBeagle 2"
+			(at 0 0 0)
+			(hide yes)
+			(effects
+				(font
+					(size 1.27 1.27)
+				)
+			)
+		)
+		(property "Mouser" "TBD"
+			(at 0 0 0)
+			(hide yes)
+			(effects
+				(font
+					(size 1.27 1.27)
+				)
+			)
+		)
+		(property "Digikey" "TBD"
+			(at 0 0 0)
+			(hide yes)
+			(effects
+				(font
+					(size 1.27 1.27)
+				)
+			)
+		)
+		(property "LCSC" "TBD"
+			(at 0 0 0)
+			(hide yes)
+			(effects
+				(font
+					(size 1.27 1.27)
+				)
+			)
+		)

Commit message: Apply signal naming convention to all nets
Connections:
- net BCLK renamed I2S_BCLK_CPU_PMOD
- net INT_N/PWRDN_N renamed INT_PWDN_N_CPU_PHY
- net LRCK renamed I2S_LRCLK_CPU_PMOD
- net MDIO0_DIO renamed MDIO_DIO_CPU_PHY
- net MDIO0_MDC renamed MDIO_MDC_CPU_PHY
- net PMOD1_SDIN renamed I2S_SDIN_CPU_to_PMOD1
- net PMOD1_SDOUT renamed I2S_SDOUT_PMOD1_to_CPU
- net PMOD2.SDIN renamed I2S_SDIN_CPU_to_PMOD2
- net PMOD2.SDOUT renamed I2S_SDOUT_PMOD2_to_CPU
- net RESET_N renamed RESET_N_CPU_to_PHY
- net RGMII_RD0 renamed RGMII_RD0_PHY_to_CPU
- net RGMII_RD1 renamed RGMII_RD1_PHY_to_CPU
- net RGMII_RD2 renamed RGMII_RD2_PHY_to_CPU
- net RGMII_RD3 renamed RGMII_RD3_PHY_to_CPU
- net RGMII_RX_CLK renamed RGMII_RX_CLK_PHY_to_CPU
- net RGMII_RX_CTRL renamed RGMII_RX_CTRL_PHY_to_CPU
- net RGMII_TD0 renamed RGMII_TD0_CPU_to_PHY
- net RGMII_TD1 renamed RGMII_TD1_CPU_to_PHY
- net RGMII_TD2 renamed RGMII_TD2_CPU_to_PHY
- net RGMII_TD3 renamed RGMII_TD3_CPU_to_PHY
- net RGMII_TX_CLK renamed RGMII_TX_CLK_CPU_to_PHY
- net RGMII_TX_CTRL renamed RGMII_TX_CTRL_CPU_to_PHY
Other:
- sheet Network ports: added INT_PWDN_N_CPU_PHY, MDIO_DIO_CPU_PHY, MDIO_MDC_CPU_PHY, RESET_N_CPU_to_PHY, RGMII_RD0_PHY_to_CPU, RGMII_RD1_PHY_to_CPU, RGMII_RD2_PHY_to_CPU, RGMII_RD3_PHY_to_CPU, RGMII_RX_CLK_PHY_to_CPU, RGMII_RX_CTRL_PHY_to_CPU, RGMII_TD0_CPU_to_PHY, RGMII_TD1_CPU_to_PHY, RGMII_TD2_CPU_to_PHY, RGMII_TD3_CPU_to_PHY, RGMII_TX_CLK_CPU_to_PHY, RGMII_TX_CTRL_CPU_to_PHY, VDD_1V1, VDD_2V5, VDD_3V3; removed 1V1, 2V5, 3V3, INT_PWDN_N, MDIO_DIO, MDIO_MDC, RGMII_RD0, RGMII_RD1, RGMII_RD2, RGMII_RD3, RGMII_RX_CLK, RGMII_RX_CTRL, RGMII_TD0, RGMII_TD1, RGMII_TD2, RGMII_TD3, RGMII_TX_CLK, RGMII_TX_CTRL, RST_N
- sheet audio ports: added I2S_BCLK_CPU_PMOD, I2S_LRCLK_CPU_PMOD, I2S_SDIN_CPU_to_PMOD1, I2S_SDIN_CPU_to_PMOD2, I2S_SDOUT_PMOD1_to_CPU, I2S_SDOUT_PMOD2_to_CPU, VDD_3V3; removed 3V3, BCLK, LRCLK, PMOD1_SDIN, PMOD1_SDOUT, PMOD2_SDIN, PMOD2_SDOUT
- sheet ldo_1v1 ports: added VDD_1V1, VDD_3V3; removed 1V1, 3V3
- sheet ldo_2v5 ports: added VDD_2V5, VDD_3V3; removed 2V5, 3V3
