File: expansion.kicad_sch (KiCad schematic)
At the start: 2 parts, among them J2 Header_18x02_2.54mm_2.54mm_St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, J3 Header_18x02_2.54mm_2.54mm_St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

Commit message: Improve schematic readability across all sheets
Other:
- note added: "Power inputs a stacked module may drive:"
