File: oscillator.kicad_sch (KiCad schematic)
At the start: 5 parts, among them Y1 ECS-2520MV-xxx-xx

Commit message: Migrate oscillator sheet to KL library symbols
Parts:
- C14, C18: value 27pf -> 27p; footprint Capacitor_SMD:C_0402_1005Metric_Pad0.74x0.62mm_HandSolder -> KL_Footprints:C_0402; symbol Device:C -> KL_C:C_27p_50V_5pct_C0G_0402; Dielectric (none) -> C0G; Digikey (none) -> TBD; LCSC (none) -> TBD; MPN (none) -> GRM1555C1H270JA01D; Mouser (none) -> 81-GRM1555C1H270JA01D; Package_in_inch (none) -> 0402; Tolerance_in_pct (none) -> 5; Voltage_in_V (none) -> 50
- C4: value 0.1uF -> 100n; footprint Capacitor_SMD:C_0402_1005Metric_Pad0.74x0.62mm_HandSolder -> KL_Footprints:C_0402; symbol Device:C -> KL_C:C_100n_35V_10pct_X7R_0402; Dielectric (none) -> X7R; Digikey (none) -> 445-6901-1-ND; LCSC (none) -> C2181802; MPN (none) -> CGA2B3X7R1V104K050BB; Mouser (none) -> 810-CGA2B3X7R1V104K; Package_in_inch (none) -> 0402; Tolerance_in_pct (none) -> 10; Voltage_in_V (none) -> 35
- TP4: value TestPoint -> TestPoint_SMD; footprint TestPoint:TestPoint_Pad_1.0x1.0mm -> KL_Footprints:TestPoint_SMD_1.0x1.0mm; symbol Connector:TestPoint -> KL_TestPoint:TestPoint_SMD
- Y1: value ECS-2520MV-xxx-xx -> 25M; footprint Oscillator:Oscillator_SMD_ECS_2520MV-xxx-xx-4Pin_2.5x2.0mm -> KL_Footprints:ECS-2520MV; symbol Oscillator:ECS-2520MV-xxx-xx -> KL_Oscillator:Oscillator_25M_25ppm_HCMOS_2.5x2.0; Digikey (none) -> TBD; Frequency_Stability_in_ppm (none) -> 25; LCSC (none) -> C405464; MPN (none) -> ECS-2520MV-250-CN-TR; Mouser (none) -> TBD; Output (none) -> HCMOS; Voltage_in_V (none) -> 1.6-3.6

Commit message: Apply signal naming convention to all nets
Connections:
- net 3V3 renamed VDD_3V3
- net X_IN renamed CLK_25M_OSC_to_PHY
Changed lines of the file:
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@@
 		)
 	)
-	(hierarchical_label "3V3"
+	(hierarchical_label "VDD_3V3"
 		(shape input)
 		(at 85.09 88.9 180)
@@
 		)
 	)
-	(label "3V3"
+	(label "VDD_3V3"
 		(at 100.33 77.47 0)
 		(effects
@@
 		)
 	)
-	(label "X_IN"
+	(label "CLK_25M_OSC_to_PHY"
 		(at 120.65 73.66 0)
 		(effects
@@
 		)
 	)
-	(hierarchical_label "X_IN"
+	(hierarchical_label "CLK_25M_OSC_to_PHY"
 		(shape output)
 		(at 133.35 73.66 0)
@@
 		)
 	)
-	(label "3V3"
+	(label "VDD_3V3"
 		(at 92.71 73.66 0)
 		(effects

Commit message: Improve schematic readability across all sheets
Other:
- moved on the sheet: C4
Changed lines of the file:
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@@
 		(dnp no)
 		(property "Reference" "Y1"
-			(at 104.14 85.09 0)
-			(effects
-				(font
-					(size 1.27 1.27)
-				)
-				(justify left)
+			(at 100.33 72.39 0)
+			(effects
+				(font
+					(size 1.27 1.27)
+				)
 			)
 		)
 		(property "Value" "25M"
-			(at 104.14 87.63 0)
-			(effects
-				(font
-					(size 1.27 1.27)
-				)
-				(justify left)
+			(at 100.33 74.93 0)
+			(effects
+				(font
+					(size 1.27 1.27)
+				)
 			)
 		)
@@
 		(property "Reference" "#PWR0920"
 			(at 104.14 95.25 0)
+			(hide yes)
 			(effects
 				(font
@@
 		)
 	)
-	(label "CLK_25M_OSC_to_PHY"
-		(at 120.65 73.66 0)
-		(effects
-			(font
-				(size 1.27 1.27)
-			)
-			(justify left bottom)
-		)
-	)
 	(hierarchical_label "CLK_25M_OSC_to_PHY"
 		(shape output)
@@
 		(property "Reference" "#PWR0921"
 			(at 129.54 82.55 0)
+			(hide yes)
 			(effects
 				(font
@@
 		(property "Value" "TestPoint_SMD"
 			(at 133.35 67.31 0)
+			(hide yes)
 			(effects
 				(font
@@
 	(symbol
 		(lib_id "KL_C:C_100n_35V_10pct_X7R_0402")
-		(at 92.71 80.01 0)
+		(at 78.74 80.01 0)
 		(unit 1)
 		(exclude_from_sim no)
@@
 	(wire
 		(pts
-			(xy 92.71 76.2) (xy 92.71 73.66)
+			(xy 78.74 76.2) (xy 78.74 73.66)
 		)
 		(stroke
@@
 	)
 	(label "VDD_3V3"
-		(at 92.71 73.66 0)
+		(at 78.74 73.66 0)
 		(effects
 			(font
@@
 	(wire
 		(pts
-			(xy 92.71 83.82) (xy 92.71 86.36)
+			(xy 78.74 83.82) (xy 78.74 86.36)
 		)
 		(stroke
@@
 	(symbol
 		(lib_id "power:GND")
-		(at 92.71 86.36 0)
+		(at 78.74 86.36 0)
 		(unit 1)
 		(exclude_from_sim no)
@@
 		(property "Reference" "#PWR0922"
 			(at 96.52 82.55 0)
-			(effects
-				(font
+			(hide yes)
+			(effects
+				(font
