File: oscillator.kicad_sch (KiCad schematic)
At the start: 5 parts, among them Y1 25M

Commit message: Migrate oscillator sheet to KiCad 10 file format
Parts:
- C14, C18: Digikey TBD -> 490-5869-1-ND; LCSC TBD -> C76961
- Y1: Digikey TBD -> XC2752TR-ND
Other:
- company: (none) -> Kebag Logic: kebag-logic.com
- title: (none) -> Oscillator

Commit message: Fix RX_CTRL and RX_D7 straps, oscillator load, RBIAS
Parts:
- C18: value 27p -> 22p; symbol KL_C:C_27p_50V_5pct_C0G_0402 -> KL_C:C_22p_50V_5pct_C0G_0402; Digikey 490-5869-1-ND -> 490-5868-1-ND; LCSC C76961 -> C76960; MPN GRM1555C1H270JA01D -> GRM1555C1H220JA01D; Mouser 81-GRM1555C1H270JA01D -> 81-GRM1555C1H220JA01D
Changed lines of the file:
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@@
 	)
 	(symbol
-		(lib_id "KL_C:C_27p_50V_5pct_C0G_0402")
+		(lib_id "KL_C:C_22p_50V_5pct_C0G_0402")
 		(at 125.73 80.01 180)
 		(unit 1)
@@
 			)
 		)
-		(property "Value" "27p"
+		(property "Value" "22p"
 			(at 129.54 60.96 0)
 			(show_name no)
@@
 			)
 		)
-		(property "Datasheet" "https://www.murata.com/en-global/products/productdetail?partno=GRM1555C1H270JA01%23"
+		(property "Datasheet" "https://www.murata.com/en-global/products/productdetail?partno=GRM1555C1H220JA01%23"
 			(at 129.54 83.82 0)
 			(hide yes)
@@
 			)
 		)
-		(property "MPN" "GRM1555C1H270JA01D"
+		(property "MPN" "GRM1555C1H220JA01D"
 			(at 0 0 0)
 			(hide yes)
@@
 			)
 		)
-		(property "Mouser" "81-GRM1555C1H270JA01D"
+		(property "Mouser" "81-GRM1555C1H220JA01D"
 			(at 0 0 0)
 			(hide yes)
@@
 			)
 		)
-		(property "Digikey" "490-5869-1-ND"
+		(property "Digikey" "490-5868-1-ND"
 			(at 0 0 0)
 			(hide yes)
@@
 			)
 		)
-		(property "LCSC" "C76961"
+		(property "LCSC" "C76960"
 			(at 0 0 0)
 			(hide yes)

Commit message: Switch BOM to in-stock LCSC parts, U3 to TLV73311
Parts:
- C14: Digikey 490-5869-1-ND -> (none); LCSC C76961 -> C1557; MPN GRM1555C1H270JA01D -> 0402CG270J500NT; Mouser 81-GRM1555C1H270JA01D -> (none)
- C4: Digikey 445-6901-1-ND -> (none); LCSC C2181802 -> C307331; MPN CGA2B3X7R1V104K050BB -> CL05B104KB54PNC; Mouser 810-CGA2B3X7R1V104K -> (none); Voltage_in_V 35 -> 50
Changed lines of the file:
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@@
 			)
 		)
-		(property "Datasheet" "https://product.tdk.com/system/files/dam/doc/product/capacitor/ceramic/mlcc/catalog/mlcc_automotive_general_en.pdf"
+		(property "Datasheet" "https://www.lcsc.com/datasheet/lcsc_datasheet_2304140030_Samsung-Electro-Mechanics-CL05B104KB54PNC_C307331.pdf"
 			(at 96.52 83.82 0)
 			(hide yes)
@@
 			)
 		)
-		(property "Voltage_in_V" "35"
+		(property "Voltage_in_V" "50"
 			(at 0 0 0)
 			(hide yes)
@@
 			)
 		)
-		(property "MPN" "CGA2B3X7R1V104K050BB"
-			(at 0 0 0)
-			(hide yes)
-			(show_name no)
-			(do_not_autoplace no)
-			(effects
-				(font
-					(size 1.27 1.27)
-				)
-			)
-		)
-		(property "Mouser" "810-CGA2B3X7R1V104K"
-			(at 0 0 0)
-			(hide yes)
-			(show_name no)
-			(do_not_autoplace no)
-			(effects
-				(font
-					(size 1.27 1.27)
-				)
-			)
-		)
-		(property "Digikey" "445-6901-1-ND"
-			(at 0 0 0)
-			(hide yes)
-			(show_name no)
-			(do_not_autoplace no)
-			(effects
-				(font
-					(size 1.27 1.27)
-				)
-			)
-		)
-		(property "LCSC" "C2181802"
+		(property "MPN" "CL05B104KB54PNC"
+			(at 0 0 0)
+			(hide yes)
+			(show_name no)
+			(do_not_autoplace no)
+			(effects
+				(font
+					(size 1.27 1.27)
+				)
+			)
+		)
+		(property "Mouser" ""
+			(at 0 0 0)
+			(hide yes)
+			(show_name no)
+			(do_not_autoplace no)
+			(effects
+				(font
+					(size 1.27 1.27)
+				)
+			)
+		)
+		(property "Digikey" ""
+			(at 0 0 0)
+			(hide yes)
+			(show_name no)
+			(do_not_autoplace no)
+			(effects
+				(font
+					(size 1.27 1.27)
+				)
+			)
+		)
+		(property "LCSC" "C307331"
 			(at 0 0 0)
 			(hide yes)
@@
 			)
 		)
-		(property "Datasheet" "https://www.murata.com/en-global/products/productdetail?partno=GRM1555C1H270JA01%23"
+		(property "Datasheet" "https://www.lcsc.com/datasheet/lcsc_datasheet_2304140030_FH--Guangdong-Fenghua-Advanced-Tech-0402CG270J500NT_C1557.pdf"
 			(at 121.92 83.82 0)
 			(hide yes)
@@
 			)
 		)
-		(property "MPN" "GRM1555C1H270JA01D"
-			(at 0 0 0)
-			(hide yes)
-			(show_name no)
-			(do_not_autoplace no)
-			(effects
-				(font
-					(size 1.27 1.27)
-				)
-			)
-		)
-		(property "Mouser" "81-GRM1555C1H270JA01D"
-			(at 0 0 0)
-			(hide yes)
-			(show_name no)
-			(do_not_autoplace no)
-			(effects
-				(font
-					(size 1.27 1.27)
-				)
-			)
-		)
-		(property "Digikey" "490-5869-1-ND"
-			(at 0 0 0)
-			(hide yes)
-			(show_name no)
-			(do_not_autoplace no)
-			(effects
-				(font
-					(size 1.27 1.27)
-				)
-			)
-		)
-		(property "LCSC" "C76961"
-			(at 0 0 0)
-			(hide yes)
+		(property "MPN" "0402CG270J500NT"
+			(at 0 0 0)
+			(hide yes)
+			(show_name no)
+			(do_not_autoplace no)
+			(effects
+				(font
+					(size 1.27 1.27)
+				)
+			)
+		)
+		(property "Mouser" ""
+			(at 0 0 0)
+			(hide yes)
+			(show_name no)
+			(do_not_autoplace no)
+			(effects
+				(font
+					(size 1.27 1.27)
+				)
+			)
+		)
+		(property "Digikey" ""
+			(at 0 0 0)
+			(hide yes)
+			(show_name no)
+			(do_not_autoplace no)
+			(effects
+				(font
+					(size 1.27 1.27)
+				)
+			)
+		)
+		(property "LCSC" "C1557"
+			(at 0 0 0)
+			(hide yes)
