File: network.kicad_sch (KiCad schematic)
At the start: 0 parts

Commit message: Migrate network sheet to KiCad 10 file format
Other:
- company: (none) -> Kebag Logic: kebag-logic.com
- title: (none) -> Network

Commit message: Add chassis isolation, remove magjack centre-tap resistor
Other:
- sheet rj45_connector_port0 ports: added none; removed VDD_2V5
Changed lines of the file:
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@@
-	(wire
-		(pts
-			(xy 127 63.5) (xy 152.4 63.5)
-		)
-		(stroke
-			(width 0)
-			(type default)
-		)
-	)
 	(wire
 		(pts
@@
 	(label "VDD_3V3"
 		(at 140.97 83.82 0)
-		(effects
-			(font
-				(size 1.27 1.27)
-			)
-			(justify left bottom)
-		)
-	)
-	(label "VDD_2V5"
-		(at 127 63.5 0)
 		(effects
 			(font
@@
 		(at 152.4 38.1)
 		(size 38.1 27.94)
+		(fields_autoplaced)
 		(exclude_from_sim no)
 		(in_bom yes)
 		(on_board yes)
 		(dnp no)
-		(fields_autoplaced yes)
 		(stroke
 			(width 0.1524)
@@
 			(effects
 				(font
-					(size 1.27 1.27)
-				)
-				(justify left)
-			)
-		)
-		(pin "VDD_2V5" input
-			(at 152.4 63.5 180)
-			(effects
-				(font
